File: kleinpad.kicad_sch (KiCad schematic)
At the start: 33 parts, among them J1 Conn_01x02, J2 Conn_01x05, SW1 RotaryEncoder_Switch, SW2 SW_Push, U1 SuperMini nRF52840

Commit message: feat: add pcb
Parts:
- removed D17, D38, D6, DI6, DI7, DI8, DS6, DS7, DS8: 1N4148, kbd:D3_TH_SMD_v2, symbol Diode:1N4148
- removed RC0-6, RC0-7, RC1-6, RC3-7: SW_Push, symbol Switch:SW_Push
- added D2, D8: 1N4148, kbd_Parts:Diode_TH_SMD, symbol Diode:1N4148
- added RC1-2, RC4-1, RC4-2: SW_Push, kbd_SW_PCBA:MX_Choc_v1v2_Hotswap_1u, symbol Switch:SW_Push
- C1, C2: value C -> 0.1u; footprint (none) -> kbd_Parts:Capacitor_1206
- D1: renamed from D16; footprint kbd:D3_TH_SMD_v2 -> kbd_Parts:Diode_TH_SMD
- D3: renamed from D26; footprint kbd:D3_TH_SMD_v2 -> kbd_Parts:Diode_TH_SMD
- D4: renamed from D27; footprint kbd:D3_TH_SMD_v2 -> kbd_Parts:Diode_TH_SMD
- D5: renamed from D36; footprint kbd:D3_TH_SMD_v2 -> kbd_Parts:Diode_TH_SMD
- D6: renamed from D37; footprint kbd:D3_TH_SMD_v2 -> kbd_Parts:Diode_TH_SMD
- D7: footprint kbd:D3_TH_SMD_v2 -> kbd_Parts:Diode_TH_SMD
- D9: renamed from D1; footprint (none) -> LED_THT:LED_D5.0mm-4_RGB
- J1: footprint (none) -> Connector_JST:JST_PH_S2B-PH-K_1x02_P2.00mm_Horizontal
- J2: footprint (none) -> Connector_PinHeader_2.54mm:PinHeader_1x05_P2.54mm_Horizontal
- OL1: footprint (none) -> kbd_Parts:OLED
- RC1-1: footprint (none) -> kbd_SW_PCBA:MX_Choc_v1v2_Hotswap_1u
- RC2-1: renamed from RC2-2; footprint (none) -> kbd_SW_PCBA:MX_Choc_v1v2_Hotswap_1u
- RC2-2: renamed from RC2-6; footprint (none) -> kbd_SW_PCBA:MX_Choc_v1v2_Hotswap_1u
- RC3-1: renamed from RC3-3; footprint (none) -> kbd_SW_PCBA:MX_Choc_v1v2_Hotswap_1u
- RC3-2: renamed from RC3-6; footprint (none) -> kbd_SW_PCBA:MX_Choc_v1v2_Hotswap_1u
- SW1: renamed from SW2; footprint (none) -> kbd_Parts:ResetSW
- SW2: renamed from SW1; footprint (none) -> Keebio-Parts.pretty-master:RotaryEncoder_EC11
Connections:
- net IO 0 is gone; now on net ROW_1: U1.17 (P0.31-LF)
- net LED_B: now also U1.12 (P1.06-LF); no longer U1.24 (P0.09-LF)
- net LED_G: now also U1.11 (P1.04-LF); no longer U1.23 (P0.10-LF)
- net LED_R: now also U1.10 (P0.11); no longer U1.22 (P1.11-LF)
- net RE_SW: now also U1.24 (P0.09-LF); no longer U1.10 (P0.11)
- net ROW_2: now reaches D4.1 (K), D6.1 (K)
- net ROW_2: now also U1.18 (P0.29-LF), D2.1 (K), D8.1 (K)
- net ROW_1: now reaches D1.1 (K), D3.1 (K), D5.1 (K)
- net ROW_1: now also D7.1 (K)
- net at D7.2 (A): now also RC4-1.2
- net INTR renamed COL_3
- net COL_3: now also RC3-1.1, RC3-2.1
- net IO 1 renamed COL_1
- net COL_1: now also U1.23 (P0.10-LF), RC1-2.1; no longer U1.18 (P0.29-LF)
- net IO 2 renamed COL_2
- net COL_2: now also U1.22 (P1.11-LF); no longer U1.19 (P0.02-LF)
- removed net IO 3: RC3-1.1, RC3-2.1, U1.20 (P1.15-LF)
- new net: D8.2 (A), RC4-2.2
- new net: D2.2 (A), RC1-2.2
- new net COL_4: RC4-1.1, RC4-2.1, U1.20 (P1.15-LF)
- no-connect marks 5 -> 4
Other:
- moved on the sheet: C1, C2, D1, D3, D4, D5, D6, D9, J1, J2, OL1, RC1-1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

Commit message: feat: 回路図を追加
Parts:
- added C3, C4: 0.1u, Capacitor_THT:C_Disc_D3.8mm_W2.6mm_P2.50mm, symbol Device:C
- added S1: RKJXV122400R, RKJXV122400R:SW_RKJXV122400R, symbol RKJXV122400R:RKJXV122400R
- C1, C2: footprint kbd_Parts:Capacitor_1206 -> Capacitor_THT:C_Disc_D3.8mm_W2.6mm_P2.50mm
- LED1: renamed from D9; footprint LED_THT:LED_D5.0mm-4_RGB -> myLibrary:LED Rectangle(OSTBMAZ2C1D); symbol Device:LED_BGKR -> Device:LED_ABGR
- RC1-1, RC1-2, RC2-1, RC2-2, RC3-1, RC3-2, RC4-1, RC4-2: footprint kbd_SW_PCBA:MX_Choc_v1v2_Hotswap_1u -> kbd_SW:CherryMX_Hotswap_1u
Connections:
- net 3V3: now also LED1.1 (A), S1.VR1_1, S1.VR2_1
- net COL_1: now also U1.12 (P1.06-LF); no longer U1.23 (P0.10-LF)
- net COL_2: now also U1.25 (P1.01-LF); no longer U1.22 (P1.11-LF)
- net COL_3: now also U1.26 (P1.02-LF); no longer U1.21 (P1.13-LF)
- net COL_4: now also U1.27 (P1.07-LF); no longer U1.20 (P1.15-LF)
- net GND: now also C3.2, C4.2, S1.B, S1.D, S1.VR1_3, S1.VR2_3; no longer LED1.3 (K)
- net LED_B: now also LED1.2 (BK), U1.19 (P0.02-LF); no longer LED1.1 (BA), U1.12 (P1.06-LF)
- net LED_G: now also LED1.3 (GK), U1.18 (P0.29-LF); no longer LED1.2 (GA), U1.11 (P1.04-LF)
- net LED_R: now also U1.17 (P0.31-LF); no longer U1.10 (P0.11)
- net MOSI: now also U1.5 (P0.17); no longer U1.7 (P0.22)
- net RE_SW: now also U1.10 (P0.11); no longer U1.24 (P0.09-LF)
- net ROW_1: now also U1.23 (P0.10-LF); no longer U1.17 (P0.31-LF)
- net ROW_2: now also U1.24 (P0.09-LF); no longer U1.18 (P0.29-LF)
- net SCK: now also U1.7 (P0.22); no longer U1.5 (P0.17)
- new net: S1.SH1 (SHIELD), S1.SH2 (SHIELD), S1.SH3 (SHIELD), S1.SH4 (SHIELD)
- new net JOY_SW: S1.A, S1.C, U1.22 (P1.11-LF)
- new net JOY_X: C3.1, S1.VR1_2, U1.21 (P1.13-LF)
- new net JOY_Y: C4.1, S1.VR2_2, U1.20 (P1.15-LF)
- no-connect marks 4 -> 2
Other:
- moved on the sheet: C1, C2, J1, J2, SW1

Commit message: fix: LEDに抵抗がない
抵抗値は手元にあるものに合わせて変更
Fixes #2
Parts:
- added R1: 100, Keebio-Parts.pretty-master:Resistor-Compact-1-side, symbol Device:R
- added R2, R3: 22, Keebio-Parts.pretty-master:Resistor-Compact-1-side, symbol Device:R
Connections:
- net LED_B: now also R3.1; no longer LED1.2 (BK)
- net LED_G: now also R2.1; no longer LED1.3 (GK)
- net LED_R: now also R1.1; no longer LED1.4 (RK)
- new net: LED1.4 (RK), R1.2
- new net: LED1.2 (BK), R3.2
- new net: LED1.3 (GK), R2.2
Other:
- moved on the sheet: LED1
